File: sdr-pager.kicad_pcb (KiCad board)
At the start: 2 copper layers, 61 x 25.4 mm, 42 parts, among them J1 Motorola Pager RF, J2 UART, J3 RF, U1 ATmega328PB, U2 Si4362, U3 24AAx, Y1 30MHz, Y2 32.768kHz

Commit message: icsp, registers
Parts:
- added TP8: SCK, TestPoint:TestPoint_Pad_1.0x1.0mm, B.Cu at (139.8, 59.6)
- added TP9: ~{RST}, TestPoint:TestPoint_Pad_1.0x1.0mm, B.Cu at (122.6, 63.4)
- C12: value 100pF -> 100nF
- C6: value 47nF -> 47uF
- TP2: value SDO -> E3
- TP3: value TX -> SDO
- TP4: value RX -> SDI
Routing:
- net GND: track 78.9 -> 104.4 mm, vias 118 -> 119
- net Net-(U1-AREF): track 0.00 -> 3.12 mm
- net ~{RESET}: track 21.8 -> 24.7 mm, vias 2 -> 3
- net I.SCK: track 23.7 -> 25.8 mm, vias 0 -> 1
- net unconnected-(U2-NC-Pad7): track 0.00 -> 1.20 mm
- net unconnected-(U2-GPIO2-Pad19): track 0.00 -> 1.20 mm
- net unconnected-(U2-NC-Pad5): track 0.00 -> 1.00 mm
- net unconnected-(U2-NC-Pad4): track 0.00 -> 0.99 mm
- net I.IRQ: track 37.3 -> 37.9 mm
- net E.SS: track 25.1 -> 24.5 mm
- net RF.VDD: track 11.3 -> 11.8 mm
Other:
- board text added: "ICSP"
