File: sdr-pager.kicad_sch (KiCad schematic)
At the start: 48 parts, among them J1 Motorola Pager RF, J2 UART, J3 RF, U1 ATmega328PB, U2 Si4362, U3 24AAx, Y1 30MHz, Y2 32.768kHz

Commit message: icsp, registers
Parts:
- added TP8: SCK, TestPoint:TestPoint_Pad_1.0x1.0mm, symbol Connector:TestPoint_Small
- added TP9: ~{RST}, TestPoint:TestPoint_Pad_1.0x1.0mm, symbol Connector:TestPoint_Small
- C12: value 100pF -> 100nF
- TP2: value SDO -> E3
- TP3: value TX -> SDO
- TP4: value RX -> SDI
Connections:
- net I.SCK: now also TP8.1
- net ~{RESET}: now also TP9.1
Changed lines of the file:
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@@
   (junction (at 125.73 182.88) (diameter 0) (color 0 0 0 0)
   )
+  (junction (at 245.11 120.65) (diameter 0) (color 0 0 0 0)
+  )
   (junction (at 58.42 83.82) (diameter 0) (color 0 0 0 0)
   )
@@
   )
   (junction (at 246.38 44.45) (diameter 0) (color 0 0 0 0)
+  )
+  (junction (at 246.38 46.99) (diameter 0) (color 0 0 0 0)
   )
   (junction (at 33.02 71.12) (diameter 0) (color 0 0 0 0)
@@
     (stroke (width 0) (type default))
   )
+  (wire (pts (xy 248.92 46.99) (xy 246.38 46.99))
+    (stroke (width 0) (type default))
+  )
   (wire (pts (xy 163.83 83.82) (xy 165.1 83.82))
     (stroke (width 0) (type default))
@@
   )
   (wire (pts (xy 205.74 86.36) (xy 213.36 86.36))
+    (stroke (width 0) (type default))
+  )
+  (wire (pts (xy 246.38 46.99) (xy 245.11 46.99))
     (stroke (width 0) (type default))
   )
@@
     )
   )
-  (global_label "I.SCK" (shape output) (at 245.11 46.99 0) (fields_autoplaced)
-    (effects (font (size 1.27 1.27)) (justify left))
-    (property "Intersheetrefs" "${INTERSHEET_REFS}" (at 253.0543 46.99 0)
+  (global_label "I.SCK" (shape output) (at 248.92 46.99 0) (fields_autoplaced)
+    (effects (font (size 1.27 1.27)) (justify left))
+    (property "Intersheetrefs" "${INTERSHEET_REFS}" (at 256.8643 46.99 0)
       (effects (font (size 1.27 1.27)) (justify left) hide)
     )
@@
       (effects (font (size 1.27 1.27)) (justify left) hide)
     )
-    (property "Value" "SDO" (at 200.66 86.36 0)
+    (property "Value" "E3" (at 200.66 86.36 0)
       (effects (font (size 1.27 1.27)) (justify left))
     )
@@
     )
   )
+  (symbol (lib_id "Connector:TestPoint_Small") (at 246.38 46.99 180) (unit 1)
+    (in_bom yes) (on_board yes) (dnp no)
+    (property "Reference" "TP8" (at 250.19 48.26 0)
+      (effects (font (size 1.27 1.27)) (justify left) hide)
+    )
+    (property "Value" "SCK" (at 260.35 46.99 0)
+      (effects (font (size 1.27 1.27)) (justify left))
+    )
+    (property "Footprint" "TestPoint:TestPoint_Pad_1.0x1.0mm" (at 241.3 46.99 0)
+      (effects (font (size 1.27 1.27)) hide)
+    )
+    (property "Datasheet" "~" (at 241.3 46.99 0)
+      (effects (font (size 1.27 1.27)) hide)
+    )
+    (pin "1")
+    (instances
+      (project "sdr-pager"
+        (path "/2ac70601-0a90-41fd-b48b-04f3b54bd23e"
+          (reference "TP8") (unit 1)
+        )
+      )
+    )
+  )
   (symbol (lib_id "power:Earth") (at 116.84 115.57 0) (unit 1)
     (in_bom yes) (on_board yes) (dnp no) (fields_autoplaced)
@@
   )
   (symbol (lib_id "Device:C_Small") (at 125.73 179.07 0) (mirror y) (unit 1)
-    (in_bom yes) (on_board yes) (dnp no) (fields_autoplaced)
-    (property "Reference" "C12" (at 123.19 177.8063 0)
-      (effects (font (size 1.27 1.27)) (justify left))
-    )
-    (property "Value" "100pF" (at 123.19 180.3463 0)
-      (effects (font (size 1.27 1.27)) (justify left))
+    (in_bom yes) (on_board yes) (dnp no)
+    (property "Reference" "C12" (at 119.38 177.8 0)
+      (effects (font (size 1.27 1.27)) (justify right))
+    )
+    (property "Value" "100nF" (at 118.11 180.34 0)
+      (effects (font (size 1.27 1.27)) (justify right))
     )
     (property "Footprint" "Capacitor_SMD:C_0603_1608Metric_Pad1.08x0.95mm_HandSolder" (at 125.73 179.07 0)
@@
       (effects (font (size 1.27 1.27)) (justify left) hide)
     )
-    (property "Value" "RX" (at 259.08 44.45 0)
+    (property "Value" "SDI" (at 260.35 44.45 0)
       (effects (font (size 1.27 1.27)) (justify left))
     )
@@
       (effects (font (size 1.27 1.27)) (justify left) hide)
     )
-    (property "Value" "TX" (at 259.08 41.91 0)
+    (property "Value" "SDO" (at 260.35 41.91 0)
       (effects (font (size 1.27 1.27)) (justify left))
     )
@@
         )
       )
+    )
+  )
+  (symbol (lib_id "Connector:TestPoint_Small") (at 245.11 120.65 180) (unit 1)
+    (in_bom yes) (on_board yes) (dnp no)
+    (property "Reference" "TP9" (at 248.92 121.92 0)
+      (effects (font (size 1.27 1.27)) (justify left) hide)
+    )
+    (property "Value" "~{RST}" (at 260.35 120.65 0)
+      (effects (font (size 1.27 1.27)) (justify left))
+    )
+    (property "Footprint" "TestPoint:TestPoint_Pad_1.0x1.0mm" (at 240.03 120.65 0)
+      (effects (font (size 1.27 1.27)) hide)
+    )
+    (property "Datasheet" "~" (at 240.03 120.65 0)
+      (effects (font (size 1.27 1.27)) hide)
+    )
+    (pin "1")
+    (instances
+      (project "sdr-pager"
+        (path "/2ac70601-0a90-41fd-b48b-04f3b54bd23e"
+          (reference "TP9") (unit 1)
+        )
+      )
